File: Hardware/KiCad/panelMeterClock/panelMeterClock.kicad_sch (KiCad schematic)
At the start: 4 parts, among them J1 DCF77 receiver, U1 ESP32-S3-WROOM-1

Commit message: intermediate commit
Parts:
- added C3, C4, C5: 10u, symbol Device:C
- added J2: PanelMeter Seconds, symbol Connector:Screw_Terminal_01x02
- added J3: PanelMeter Minutes, symbol Connector:Screw_Terminal_01x02
- added J4: PanelMeter Hours, symbol Connector:Screw_Terminal_01x02
- added R1, R3, R5: 1K, symbol Device:R
- added R2, R4, R6: 2K, symbol Device:R
Connections:
- net GND: now also C3.2, C4.2, C5.2, J2.2 (Pin_2), J3.2 (Pin_2), J4.2 (Pin_2)
- net METER_SEC: now reaches U1.10 (GPIO17/U1TXD/ADC2_CH6)
- net METER_SEC: now also R1.1
- net METER_HOUR: now reaches U1.8 (GPIO15/U0RTS/ADC2_CH4/XTAL_32K_P)
- net METER_HOUR: now also R5.1
- net METER_MIN: now reaches U1.9 (GPIO16/U0CTS/ADC2_CH5/XTAL_32K_N)
- net METER_MIN: now also R3.1
- new net: C5.1, R5.2, R6.1
- new net: J4.1 (Pin_1), R6.2
- new net: J3.1 (Pin_1), R4.2
- new net: C3.1, R1.2, R2.1
- new net: J2.1 (Pin_1), R2.2
- new net: C4.1, R3.2, R4.1
